File: hardware/pcb/power.kicad_sch (KiCad schematic)
At the start: 40 parts, among them J1 USB-C Port B, J2 USB-C Port A, U1 USBLC6-2SC6, U2 USBLC6-2SC6, U3 TPS2121RUX, U4 TPS22965DSG, U5 AP2127N-3.3

Commit message: Add audio, microSD and keyboard I2C, and place parts on the PCB
Schematics:
- Swap the MAX98357A for the TLV320DAC3100 (headphone and speaker out).
  A 12 MHz oscillator drives MCLK and the codec is the I2S clock master,
  so the stock simple-audio-card works without a custom machine driver.
- Add the microSD slot for the CM0Lite; the SD pull-ups are footprints only.
- Add HID over I2C from the RP2040 to the CM0 (KB_SDA/KB_SCL/KB_INT) on
  i2c-gpio, so the keyboard works on stock Raspberry Pi OS. Add test pads.
- Use power symbols for +1V1, assign footprints and LCSC numbers, and
  fix global label shapes.

PCB: 228.6 x 146.2 mm outline and a provisional bottom-side placement,
with HID USB top-left and Linux USB top-right. Add footprints for the CM0,
TPS2121 (RUX), the 22-pin DSI FPC and the CR2032 holder.

Docs: record the decisions and open items. Add a draft device tree
overlay for the audio codec.

Co-Authored-By: Claude Opus 5.5 <noreply@anthropic.com>
Parts:
- C4: footprint (none) -> Capacitor_SMD:CP_Elec_6.3x7.7; LCSC (none) -> C46550459
- TP1, TP2, TP3, TP4, TP5, TP6, TP7: footprint (none) -> TestPoint:TestPoint_Pad_D1.5mm
- U3: footprint (none) -> Skjar:Texas_RUX_VQFN-HR-12_2.5x2mm_P0.5mm
- U4: footprint (none) -> Package_SON:Texas_DSG0008A_WSON-8-1EP_2x2mm_P0.5mm_EP0.9x1.6mm
