File: hardware/pcb/keymatrix.kicad_sch (KiCad schematic)
At the start: 0 parts

Commit message: Add 42-key matrix sheet, layout, and USB-C part
- Key layout from Smidr (KLE format, 42 keys) in hardware/layout,
  with the 7x6 COL2ROW matrix mapping proven on the blad keyboard
- Keymatrix sheet: 42 Choc hotswap switches and 1N4148W diodes
  (C81598, Basic), every pin labeled; RP2040 ROW/COL nets are now
  global labels, GPIO13/14 freed as spares
- USB-C receptacles J1/J2 set to HRO TYPE-C-31-M-12 (C165948)
- Power sheet: CC lines reach the RP2040 ADC again
- Docs: design decisions, pin assignment, keymatrix spec and
  reference, open items

Full project netlist matches all 141 intended nets; ERC has no errors.

Co-Authored-By: Claude Opus 5.5 <noreply@anthropic.com>
Parts:
- added D501, D502, D503, D504, D505, D506, D507, D508, D509, D510, D511, D512, D513, D514, D515, D516, D517, D518, D519, D520, D521, D522, D523, D524, D525, D526, D527, D528, D529, D530, D531, D532, D533, D534, D535, D536, D537, D538, D539, D540, D541, D542: 1N4148W, Diode_SMD:D_SOD-123, symbol Device:D
- added SW501: Esc, Skjar:SW_Kailh_Choc_Hotswap, symbol Switch:SW_Push
- added SW502: Q, Skjar:SW_Kailh_Choc_Hotswap, symbol Switch:SW_Push
- added SW503: W, Skjar:SW_Kailh_Choc_Hotswap, symbol Switch:SW_Push
- added SW504: E, Skjar:SW_Kailh_Choc_Hotswap, symbol Switch:SW_Push
- added SW505: R, Skjar:SW_Kailh_Choc_Hotswap, symbol Switch:SW_Push
- added SW506: T, Skjar:SW_Kailh_Choc_Hotswap, symbol Switch:SW_Push
- added SW507: Y, Skjar:SW_Kailh_Choc_Hotswap, symbol Switch:SW_Push
- added SW508: U, Skjar:SW_Kailh_Choc_Hotswap, symbol Switch:SW_Push
- added SW509: I, Skjar:SW_Kailh_Choc_Hotswap, symbol Switch:SW_Push
- added SW510: O, Skjar:SW_Kailh_Choc_Hotswap, symbol Switch:SW_Push
- added SW511: P, Skjar:SW_Kailh_Choc_Hotswap, symbol Switch:SW_Push
- added SW512: Bksp, Skjar:SW_Kailh_Choc_Hotswap, symbol Switch:SW_Push
- added SW513: Tab, Skjar:SW_Kailh_Choc_Hotswap, symbol Switch:SW_Push
- added SW514: A, Skjar:SW_Kailh_Choc_Hotswap, symbol Switch:SW_Push
- added SW515: S, Skjar:SW_Kailh_Choc_Hotswap, symbol Switch:SW_Push
- added SW516: D, Skjar:SW_Kailh_Choc_Hotswap, symbol Switch:SW_Push
- added SW517: F, Skjar:SW_Kailh_Choc_Hotswap, symbol Switch:SW_Push
- added SW518: G, Skjar:SW_Kailh_Choc_Hotswap, symbol Switch:SW_Push
- added SW519: H, Skjar:SW_Kailh_Choc_Hotswap, symbol Switch:SW_Push
- added SW520: J, Skjar:SW_Kailh_Choc_Hotswap, symbol Switch:SW_Push
- added SW521: K, Skjar:SW_Kailh_Choc_Hotswap, symbol Switch:SW_Push
- added SW522: L, Skjar:SW_Kailh_Choc_Hotswap, symbol Switch:SW_Push
- added SW523: Enter, Skjar:SW_Kailh_Choc_Hotswap, symbol Switch:SW_Push
- added SW524: LShift, Skjar:SW_Kailh_Choc_Hotswap, symbol Switch:SW_Push
- added SW525: Z, Skjar:SW_Kailh_Choc_Hotswap, symbol Switch:SW_Push
- added SW526: X, Skjar:SW_Kailh_Choc_Hotswap, symbol Switch:SW_Push
- added SW527: C, Skjar:SW_Kailh_Choc_Hotswap, symbol Switch:SW_Push
- added SW528: V, Skjar:SW_Kailh_Choc_Hotswap, symbol Switch:SW_Push
- added SW529: B, Skjar:SW_Kailh_Choc_Hotswap, symbol Switch:SW_Push
- added SW530: N, Skjar:SW_Kailh_Choc_Hotswap, symbol Switch:SW_Push
- added SW531: M, Skjar:SW_Kailh_Choc_Hotswap, symbol Switch:SW_Push
- added SW532: <, Skjar:SW_Kailh_Choc_Hotswap, symbol Switch:SW_Push
- added SW533: >, Skjar:SW_Kailh_Choc_Hotswap, symbol Switch:SW_Push
- added SW534: ?, Skjar:SW_Kailh_Choc_Hotswap, symbol Switch:SW_Push
- added SW535: LCtrl, Skjar:SW_Kailh_Choc_Hotswap, symbol Switch:SW_Push
- added SW536: LGui, Skjar:SW_Kailh_Choc_Hotswap, symbol Switch:SW_Push
- added SW537: LAlt, Skjar:SW_Kailh_Choc_Hotswap, symbol Switch:SW_Push
- added SW538, SW539: Space, Skjar:SW_Kailh_Choc_Hotswap, symbol Switch:SW_Push
- added SW540: RAlt, Skjar:SW_Kailh_Choc_Hotswap, symbol Switch:SW_Push
- added SW541: RGui, Skjar:SW_Kailh_Choc_Hotswap, symbol Switch:SW_Push
- added SW542: RCtrl, Skjar:SW_Kailh_Choc_Hotswap, symbol Switch:SW_Push
Connections:
- new net COL0: SW501.1, SW512.1, SW513.1, SW524.1, SW535.1, SW541.1, SW542.1
- new net COL1: SW502.1, SW511.1, SW514.1, SW523.1, SW525.1, SW534.1, SW536.1
- new net COL2: SW503.1, SW510.1, SW515.1, SW522.1, SW526.1, SW533.1, SW537.1
- new net COL3: SW504.1, SW509.1, SW516.1, SW521.1, SW527.1, SW532.1, SW540.1
- new net COL4: SW505.1, SW508.1, SW517.1, SW520.1, SW528.1, SW531.1, SW538.1
- new net COL5: SW506.1, SW507.1, SW518.1, SW519.1, SW529.1, SW530.1, SW539.1
- new net ROW0: D501.1 (K), D502.1 (K), D503.1 (K), D504.1 (K), D505.1 (K), D506.1 (K)
- new net ROW1: D507.1 (K), D508.1 (K), D509.1 (K), D510.1 (K), D511.1 (K), D512.1 (K)
- new net ROW2: D513.1 (K), D514.1 (K), D515.1 (K), D516.1 (K), D517.1 (K), D518.1 (K)
- new net ROW3: D519.1 (K), D520.1 (K), D521.1 (K), D522.1 (K), D523.1 (K), D542.1 (K)
- new net ROW4: D524.1 (K), D525.1 (K), D526.1 (K), D527.1 (K), D528.1 (K), D529.1 (K)
- new net ROW5: D530.1 (K), D531.1 (K), D532.1 (K), D533.1 (K), D534.1 (K), D541.1 (K)
- new net ROW6: D535.1 (K), D536.1 (K), D537.1 (K), D538.1 (K), D539.1 (K), D540.1 (K)
- new net SW10_D: D510.2 (A), SW510.2
- new net SW11_D: D511.2 (A), SW511.2
- new net SW12_D: D512.2 (A), SW512.2
- new net SW13_D: D513.2 (A), SW513.2
- new net SW14_D: D514.2 (A), SW514.2
- new net SW15_D: D515.2 (A), SW515.2
- new net SW16_D: D516.2 (A), SW516.2
- new net SW17_D: D517.2 (A), SW517.2
- new net SW18_D: D518.2 (A), SW518.2
- new net SW19_D: D519.2 (A), SW519.2
- new net SW1_D: D501.2 (A), SW501.2
- new net SW20_D: D520.2 (A), SW520.2
- new net SW21_D: D521.2 (A), SW521.2
- new net SW22_D: D522.2 (A), SW522.2
- new net SW23_D: D523.2 (A), SW523.2
- new net SW24_D: D524.2 (A), SW524.2
- new net SW25_D: D525.2 (A), SW525.2
- new net SW26_D: D526.2 (A), SW526.2
- new net SW27_D: D527.2 (A), SW527.2
- new net SW28_D: D528.2 (A), SW528.2
- new net SW29_D: D529.2 (A), SW529.2
- new net SW2_D: D502.2 (A), SW502.2
- new net SW30_D: D530.2 (A), SW530.2
- new net SW31_D: D531.2 (A), SW531.2
- new net SW32_D: D532.2 (A), SW532.2
- new net SW33_D: D533.2 (A), SW533.2
- new net SW34_D: D534.2 (A), SW534.2
- new net SW35_D: D535.2 (A), SW535.2
- new net SW36_D: D536.2 (A), SW536.2
- new net SW37_D: D537.2 (A), SW537.2
- new net SW38_D: D538.2 (A), SW538.2
- new net SW39_D: D539.2 (A), SW539.2
- new net SW3_D: D503.2 (A), SW503.2
- new net SW40_D: D540.2 (A), SW540.2
- new net SW41_D: D541.2 (A), SW541.2
- new net SW42_D: D542.2 (A), SW542.2
- new net SW4_D: D504.2 (A), SW504.2
- new net SW5_D: D505.2 (A), SW505.2
- new net SW6_D: D506.2 (A), SW506.2
- new net SW7_D: D507.2 (A), SW507.2
- new net SW8_D: D508.2 (A), SW508.2
- new net SW9_D: D509.2 (A), SW509.2
Other:
- note added: "キーマトリクス（7 行 × 6 列、COL2ROW。対応は hardware/layout/README.md）"
- title: (none) -> SKJÁR Key matrix

Commit message: Add per-key RGB, finish schematic wiring, and document HID over I2C
- Add SK6812MINI-E per-key RGB with a switched +5V_LED rail and an
  AHCT buffer on the data line; remove SW102 to free GPIO20
- Use D_Small for the matrix diodes and replace labels with wires
- Tidy the keymatrix sheet layout without changing connectivity
- Document the HID over I2C keyboard path, back-power rules and
  role split across README and docs

Co-Authored-By: Claude Opus 5.5 <noreply@anthropic.com>
Parts:
- added C501, C502, C503, C504, C505, C506, C507, C508, C509, C510, C511, C512, C513, C514, C515, C516, C517, C518, C519, C520, C521, C522, C523, C524, C525, C526, C527, C528, C529, C530, C531, C532, C533, C534, C535, C536, C537, C538, C539, C540, C541, C542, C544, C545: 100n, Capacitor_SMD:C_0603_1608Metric, symbol Device:C
- added C543: 10u, Capacitor_SMD:C_0603_1608Metric, symbol Device:C
- added LED501, LED502, LED503, LED504, LED505, LED506, LED507, LED508, LED509, LED510, LED511, LED512, LED513, LED514, LED515, LED516, LED517, LED518, LED519, LED520, LED521, LED522, LED523, LED524, LED525, LED526, LED527, LED528, LED529, LED530, LED531, LED532, LED533, LED534, LED535, LED536, LED537, LED538, LED539, LED540, LED541, LED542: SK6812MINI-E, LED_SMD:LED_SK6812MINI-E_3.2x2.8mm_P1.5mm_ReverseMount, symbol LED:SK6812MINI-E
- added Q501: AO3401A, Package_TO_SOT_SMD:SOT-23, symbol Transistor_FET:AO3401A
- added Q502: 2N7002, Package_TO_SOT_SMD:SOT-23, symbol Transistor_FET:2N7002
- added R501, R503: 100k, Resistor_SMD:R_0603_1608Metric, symbol Device:R
- added R502: 10k, Resistor_SMD:R_0603_1608Metric, symbol Device:R
- added R504: 330, Resistor_SMD:R_0603_1608Metric, symbol Device:R
- added U501: 74AHCT1G125, Package_TO_SOT_SMD:SOT-23-5, symbol 74xGxx:74AHCT1G125
- D501, D502, D503, D504, D505, D506, D507, D508, D509, D510, D511, D512, D513, D514, D515, D516, D517, D518, D519, D520, D521, D522, D523, D524, D525, D526, D527, D528, D529, D530, D531, D532, D533, D534, D535, D536, D537, D538, D539, D540, D541, D542: symbol Device:D -> Device:D_Small
Connections:
- net SW10_D: no longer names the net of D510.2 (A), SW510.2
- net SW11_D: no longer names the net of D511.2 (A), SW511.2
- net SW12_D: no longer names the net of D512.2 (A), SW512.2
- net SW13_D: no longer names the net of D513.2 (A), SW513.2
- net SW14_D: no longer names the net of D514.2 (A), SW514.2
- net SW15_D: no longer names the net of D515.2 (A), SW515.2
- net SW16_D: no longer names the net of D516.2 (A), SW516.2
- net SW17_D: no longer names the net of D517.2 (A), SW517.2
- net SW18_D: no longer names the net of D518.2 (A), SW518.2
- net SW19_D: no longer names the net of D519.2 (A), SW519.2
- net SW1_D: no longer names the net of D501.2 (A), SW501.2
- net SW20_D: no longer names the net of D520.2 (A), SW520.2
- net SW21_D: no longer names the net of D521.2 (A), SW521.2
- net SW22_D: no longer names the net of D522.2 (A), SW522.2
- net SW23_D: no longer names the net of D523.2 (A), SW523.2
- net SW24_D: no longer names the net of D524.2 (A), SW524.2
- net SW25_D: no longer names the net of D525.2 (A), SW525.2
- net SW26_D: no longer names the net of D526.2 (A), SW526.2
- net SW27_D: no longer names the net of D527.2 (A), SW527.2
- net SW28_D: no longer names the net of D528.2 (A), SW528.2
- net SW29_D: no longer names the net of D529.2 (A), SW529.2
- net SW2_D: no longer names the net of D502.2 (A), SW502.2
- net SW30_D: no longer names the net of D530.2 (A), SW530.2
- net SW31_D: no longer names the net of D531.2 (A), SW531.2
- net SW32_D: no longer names the net of D532.2 (A), SW532.2
- net SW33_D: no longer names the net of D533.2 (A), SW533.2
- net SW34_D: no longer names the net of D534.2 (A), SW534.2
- net SW35_D: no longer names the net of D535.2 (A), SW535.2
- net SW36_D: no longer names the net of D536.2 (A), SW536.2
- net SW37_D: no longer names the net of D537.2 (A), SW537.2
- net SW38_D: no longer names the net of D538.2 (A), SW538.2
- net SW39_D: no longer names the net of D539.2 (A), SW539.2
- net SW3_D: no longer names the net of D503.2 (A), SW503.2
- net SW40_D: no longer names the net of D540.2 (A), SW540.2
- net SW41_D: no longer names the net of D541.2 (A), SW541.2
- net SW42_D: no longer names the net of D542.2 (A), SW542.2
- net SW4_D: no longer names the net of D504.2 (A), SW504.2
- net SW5_D: no longer names the net of D505.2 (A), SW505.2
- net SW6_D: no longer names the net of D506.2 (A), SW506.2
- net SW7_D: no longer names the net of D507.2 (A), SW507.2
- net SW8_D: no longer names the net of D508.2 (A), SW508.2
- net SW9_D: no longer names the net of D509.2 (A), SW509.2
- new net: LED509.4 (DOUT), LED510.2 (DIN)
- new net: LED510.4 (DOUT), LED511.2 (DIN)
- new net: LED524.4 (DOUT), LED525.2 (DIN)
- new net: LED525.4 (DOUT), LED526.2 (DIN)
- new net: LED504.4 (DOUT), LED505.2 (DIN)
- new net: LED505.4 (DOUT), LED506.2 (DIN)
- new net: LED541.2 (DIN), LED542.4 (DOUT)
- new net: LED540.2 (DIN), LED541.4 (DOUT)
- new net: LED506.4 (DOUT), LED507.2 (DIN)
- new net: LED508.4 (DOUT), LED509.2 (DIN)
- new net: LED521.2 (DIN), LED522.4 (DOUT)
- new net: LED520.2 (DIN), LED521.4 (DOUT)
- new net: LED511.4 (DOUT), LED512.2 (DIN)
- new net: LED512.4 (DOUT), LED523.2 (DIN)
- new net: LED519.2 (DIN), LED520.4 (DOUT)
- new net: LED518.2 (DIN), LED519.4 (DOUT)
- new net: LED522.2 (DIN), LED523.4 (DOUT)
- new net: LED535.2 (DIN), LED536.4 (DOUT)
- new net: LED502.4 (DOUT), LED503.2 (DIN)
- new net: LED503.4 (DOUT), LED504.2 (DIN)
- new net: LED501.4 (DOUT), LED502.2 (DIN)
- new net: LED507.4 (DOUT), LED508.2 (DIN)
- new net: C545.2, Q501.1 (G), R501.2, R502.2
- new net: LED517.2 (DIN), LED518.4 (DOUT)
- new net: Q502.3 (D), R502.1
- new net: LED539.2 (DIN), LED540.4 (DOUT)
- new net: LED538.2 (DIN), LED539.4 (DOUT)
- new net: LED526.4 (DOUT), LED527.2 (DIN)
- new net: LED527.4 (DOUT), LED528.2 (DIN)
- new net: LED528.4 (DOUT), LED529.2 (DIN)
- new net: LED516.2 (DIN), LED517.4 (DOUT)
- new net: R504.1, U501.4
- new net: LED515.2 (DIN), LED516.4 (DOUT)
- new net: LED529.4 (DOUT), LED530.2 (DIN)
- new net: LED530.4 (DOUT), LED531.2 (DIN)
- new net: LED536.2 (DIN), LED537.4 (DOUT)
- new net: LED531.4 (DOUT), LED532.2 (DIN)
- new net: LED532.4 (DOUT), LED533.2 (DIN)
- new net: LED533.4 (DOUT), LED534.2 (DIN)
- new net: LED534.4 (DOUT), LED542.2 (DIN)
- new net: LED513.2 (DIN), LED514.4 (DOUT)
- new net: LED513.4 (DOUT), LED524.2 (DIN)
- new net: LED514.2 (DIN), LED515.4 (DOUT)
- new net: LED537.2 (DIN), LED538.4 (DOUT)
- new net +5V: C545.1, Q501.2 (S), R501.1
- new net +5V_LED: C501.1, C502.1, C503.1, C504.1, C505.1, C506.1, C507.1, C508.1, C509.1, C510.1, C511.1, C512.1, C513.1, C514.1, C515.1, C516.1, C517.1, C518.1, C519.1, C520.1, C521.1, C522.1, C523.1, C524.1, C525.1, C526.1, C527.1, C528.1, C529.1, C530.1, C531.1, C532.1, C533.1, C534.1, C535.1, C536.1, C537.1, C538.1, C539.1, C540.1, C541.1, C542.1, C543.1, C544.1, LED501.3 (VDD), LED502.3 (VDD), LED503.3 (VDD), LED504.3 (VDD), LED505.3 (VDD), LED506.3 (VDD), LED507.3 (VDD), LED508.3 (VDD), LED509.3 (VDD), LED510.3 (VDD), LED511.3 (VDD), LED512.3 (VDD), LED513.3 (VDD), LED514.3 (VDD), LED515.3 (VDD), LED516.3 (VDD), LED517.3 (VDD), LED518.3 (VDD), LED519.3 (VDD), LED520.3 (VDD), LED521.3 (VDD), LED522.3 (VDD), LED523.3 (VDD), LED524.3 (VDD), LED525.3 (VDD), LED526.3 (VDD), LED527.3 (VDD), LED528.3 (VDD), LED529.3 (VDD), LED530.3 (VDD), LED531.3 (VDD), LED532.3 (VDD), LED533.3 (VDD), LED534.3 (VDD), LED535.3 (VDD), LED536.3 (VDD), LED537.3 (VDD), LED538.3 (VDD), LED539.3 (VDD), LED540.3 (VDD), LED541.3 (VDD), LED542.3 (VDD), Q501.3 (D), U501.5 (VCC)
- new net GND: C501.2, C502.2, C503.2, C504.2, C505.2, C506.2, C507.2, C508.2, C509.2, C510.2, C511.2, C512.2, C513.2, C514.2, C515.2, C516.2, C517.2, C518.2, C519.2, C520.2, C521.2, C522.2, C523.2, C524.2, C525.2, C526.2, C527.2, C528.2, C529.2, C530.2, C531.2, C532.2, C533.2, C534.2, C535.2, C536.2, C537.2, C538.2, C539.2, C540.2, C541.2, C542.2, C543.2, C544.2, LED501.1 (VSS), LED502.1 (VSS), LED503.1 (VSS), LED504.1 (VSS), LED505.1 (VSS), LED506.1 (VSS), LED507.1 (VSS), LED508.1 (VSS), LED509.1 (VSS), LED510.1 (VSS), LED511.1 (VSS), LED512.1 (VSS), LED513.1 (VSS), LED514.1 (VSS), LED515.1 (VSS), LED516.1 (VSS), LED517.1 (VSS), LED518.1 (VSS), LED519.1 (VSS), LED520.1 (VSS), LED521.1 (VSS), LED522.1 (VSS), LED523.1 (VSS), LED524.1 (VSS), LED525.1 (VSS), LED526.1 (VSS), LED527.1 (VSS), LED528.1 (VSS), LED529.1 (VSS), LED530.1 (VSS), LED531.1 (VSS), LED532.1 (VSS), LED533.1 (VSS), LED534.1 (VSS), LED535.1 (VSS), LED536.1 (VSS), LED537.1 (VSS), LED538.1 (VSS), LED539.1 (VSS), LED540.1 (VSS), LED541.1 (VSS), LED542.1 (VSS), Q502.2 (S), R503.2, U501.1, U501.3 (GND)
- new net RGB_D0: LED501.2 (DIN), R504.2
- new net RGB_DATA: U501.2
- new net RGB_EN: Q502.1 (G), R503.1
- no-connect marks 0 -> 1
Other:
- note added: "キーの RGB（SK6812MINI-E ×42）。詳細は docs/schematic/keymatrix.md"
- note added: "キーの RGB：LED の電源の ON / OFF とデータのバッファ"
- moved on the sheet: D501, D502, D503, D504, D505, D506, D507, D508, D509, D510, D511, D512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
